File: PCB_June/PCB.kicad_sch (KiCad schematic)
At the start: 25 parts, among them J201 FH34SRJ-24S-0.5SH_99_, Q201 BSS138, Q202 S8050, U203 AO3401

Commit message: hhhhh
Parts:
- removed C12, C13, C14, C15, C16, C17, C18, C19: 1u, Capacitor_SMD:C_0805_2012Metric_Pad1.18x1.45mm_HandSolder, symbol Device:C
- removed J201: FH34SRJ-24S-0.5SH_99_, Custom:FH34SRJ24S05SH99, symbol FH34SRJ-24S-0.5SH(99):FH34SRJ-24S-0.5SH_99_
- added C220, C221, C222, C223, C224 (x2), C226, C227: 1u, Capacitor_SMD:C_0805_2012Metric_Pad1.18x1.45mm_HandSolder, symbol Device:C
- added J202: FH34SRJ-24S-0.5SH_99_, Custom:FH34SRJ24S05SH99, symbol FH34SRJ-24S-0.5SH(99):FH34SRJ-24S-0.5SH_99_
- Q202: footprint Package_TO_SOT_SMD:SOT-23-3 -> Package_TO_SOT_THT:TO-92_Inline
Connections:
- net 3V3_OUT: now also C221.1, J202.15, J202.16
- net BS: now also C220.2, C221.2, C222.2, C223.2, C224.2, C224.2, C226.2, C227.2, J202.17, J202.8, J202.MP1, J202.MP2
- net EPD_BUSY: now also J202.9
- net EPD_CS: now also J202.12
- net EPD_DC: now also J202.11
- net EPD_DIN: now also J202.14
- net EPD_RST: now also J202.10
- net EPD_SCK: now also J202.13
- net GDR: now also J202.2
- net RESE: now also J202.3
- net VGH: now also C224.1, J202.21
- net VGL: now also C226.1, J202.23
- new net: C222.1, J202.18
- new net: C223.1, J202.20
- new net: C224.1, J202.22
- new net: C227.1, J202.24
- new net: C220.1, J202.5

Commit message: annotate
Parts:
- renumbered C221 to C10, C222 to C11, C223 to C12, C224 to C13, C224 to C14, C226 to C15, C227 to C16, C203 to C17, C201 to C7, C202 to C8, C220 to C9, D201 to D1, D202 to D2, D203 to D3, J202 to J2, L201 to L1, Q201 to Q1, Q202 to Q2, R201 to R1, R202 to R2, R204 to R3, R205 to R4, R203 to R5, R206 to R6, U203 to U3
Changed lines of the file:
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@@
 		(dnp no)
 		(fields_autoplaced yes)
-		(property "Reference" "R201"
+		(property "Reference" "R1"
 			(at 29.21 16.51 90)
 			(effects
@@
 				(path "/4d36fe0e-b49e-45a2-8e76-66c0323912e5"
 					(reference "R201")
+					(unit 1)
+				)
+			)
+			(project "EE 447"
+				(path "/8dcae476-bf02-4dea-8567-670805b7ab7c/9f33d424-8f8c-499b-911f-2b5f72ba0270"
+					(reference "R1")
 					(unit 1)
 				)
@@
 		(on_board yes)
 		(dnp no)
-		(property "Reference" "J202"
+		(property "Reference" "J2"
 			(at 40.64 168.91 0)
 			(effects
@@
 				)
 			)
+			(project "EE 447"
+				(path "/8dcae476-bf02-4dea-8567-670805b7ab7c/9f33d424-8f8c-499b-911f-2b5f72ba0270"
+					(reference "J2")
+					(unit 1)
+				)
+			)
 		)
 	)
@@
 		(on_board yes)
 		(dnp no)
-		(property "Reference" "C227"
+		(property "Reference" "C16"
 			(at 83.058 161.29 90)
 			(effects
@@
 				)
 			)
+			(project "EE 447"
+				(path "/8dcae476-bf02-4dea-8567-670805b7ab7c/9f33d424-8f8c-499b-911f-2b5f72ba0270"
+					(reference "C16")
+					(unit 1)
+				)
+			)
 		)
 	)
@@
 		(on_board yes)
 		(dnp no)
-		(property "Reference" "C221"
+		(property "Reference" "C10"
 			(at 83.058 138.43 90)
 			(effects
@@
 				)
 			)
+			(project "EE 447"
+				(path "/8dcae476-bf02-4dea-8567-670805b7ab7c/9f33d424-8f8c-499b-911f-2b5f72ba0270"
+					(reference "C10")
+					(unit 1)
+				)
+			)
 		)
 	)
@@
 		(dnp no)
 		(fields_autoplaced yes)
-		(property "Reference" "C201"
+		(property "Reference" "C7"
 			(at 29.21 43.18 90)
 			(effects
@@
 				)
 			)
+			(project "EE 447"
+				(path "/8dcae476-bf02-4dea-8567-670805b7ab7c/9f33d424-8f8c-499b-911f-2b5f72ba0270"
+					(reference "C7")
+					(unit 1)
+				)
+			)
 		)
 	)
@@
 		(dnp no)
 		(fields_autoplaced yes)
-		(property "Reference" "R203"
+		(property "Reference" "R5"
 			(at 110.49 31.7499 0)
 			(effects
@@
 				)
 			)
+			(project "EE 447"
+				(path "/8dcae476-bf02-4dea-8567-670805b7ab7c/9f33d424-8f8c-499b-911f-2b5f72ba0270"
+					(reference "R5")
+					(unit 1)
+				)
+			)
 		)
 	)
@@
 		(dnp no)
 		(fields_autoplaced yes)
-		(property "Reference" "C202"
+		(property "Reference" "C8"
 			(at 44.45 57.15 90)
 			(effects
@@
 				)
 			)
+			(project "EE 447"
+				(path "/8dcae476-bf02-4dea-8567-670805b7ab7c/9f33d424-8f8c-499b-911f-2b5f72ba0270"
+					(reference "C8")
+					(unit 1)
+				)
+			)
 		)
 	)
@@
 		(on_board yes)
 		(dnp no)
-		(property "Reference" "C223"
+		(property "Reference" "C12"
 			(at 83.058 151.13 90)
 			(effects
@@
 				)
 			)
+			(project "EE 447"
+				(path "/8dcae476-bf02-4dea-8567-670805b7ab7c/9f33d424-8f8c-499b-911f-2b5f72ba0270"
+					(reference "C12")
+					(unit 1)
+				)
+			)
 		)
 	)
@@
 		(on_board yes)
 		(dnp no)
-		(property "Reference" "D203"
+		(property "Reference" "D3"
 			(at 57.404 72.898 90)
 			(effects
@@
 				)
 			)
+			(project "EE 447"
+				(path "/8dcae476-bf02-4dea-8567-670805b7ab7c/9f33d424-8f8c-499b-911f-2b5f72ba0270"
+					(reference "D3")
+					(unit 1)
+				)
+			)
 		)
 	)
@@
 		(on_board yes)
 		(dnp no)
-		(property "Reference" "C222"
+		(property "Reference" "C11"
 			(at 83.058 146.05 90)
 			(effects
@@
 				)
 			)
+			(project "EE 447"
+				(path "/8dcae476-bf02-4dea-8567-670805b7ab7c/9f33d424-8f8c-499b-911f-2b5f72ba0270"
+					(reference "C11")
+					(unit 1)
+				)
+			)
 		)
 	)
@@
 		(on_board yes)
 		(dnp no)
-		(property "Reference" "R205"
+		(property "Reference" "R4"
 			(at 104.14 54.61 90)
 			(effects
@@
 				)
 			)
+			(project "EE 447"
+				(path "/8dcae476-bf02-4dea-8567-670805b7ab7c/9f33d424-8f8c-499b-911f-2b5f72ba0270"
+					(reference "R4")
+					(unit 1)
+				)
+			)
 		)
 	)
@@
 		(dnp no)
 		(fields_autoplaced yes)
-		(property "Reference" "D202"
+		(property "Reference" "D2"
 			(at 39.37 72.0724 90)
 			(effects
@@
 				)
 			)
+			(project "EE 447"
+				(path "/8dcae476-bf02-4dea-8567-670805b7ab7c/9f33d424-8f8c-499b-911f-2b5f72ba0270"
+					(reference "D2")
+					(unit 1)
+				)
+			)
 		)
 	)
@@
 		(dnp no)
 		(fields_autoplaced yes)
-		(property "Reference" "Q202"
+		(property "Reference" "Q2"
 			(at 124.46 46.9899 0)
 			(effects
@@
 				)
 			)
+			(project "EE 447"
+				(path "/8dcae476-bf02-4dea-8567-670805b7ab7c/9f33d424-8f8c-499b-911f-2b5f72ba0270"
+					(reference "Q2")
+					(unit 1)
+				)
+			)
 		)
 	)
@@
 		(on_board yes)
 		(dnp no)
-		(property "Reference" "C224"
+		(property "Reference" "C14"
 			(at 83.058 156.21 90)
 			(effects
@@
 				)
 			)
+			(project "EE 447"
+				(path "/8dcae476-bf02-4dea-8567-670805b7ab7c/9f33d424-8f8c-499b-911f-2b5f72ba0270"
+					(reference "C14")
+					(unit 1)
+				)
+			)
 		)
 	)
@@
 		(on_board yes)
 		(dnp no)
-		(property "Reference" "C220"
+		(property "Reference" "C9"
 			(at 81.788 113.03 90)
 			(effects
@@
 				)
 			)
+			(project "EE 447"
+				(path "/8dcae476-bf02-4dea-8567-670805b7ab7c/9f33d424-8f8c-499b-911f-2b5f72ba0270"
+					(reference "C9")
+					(unit 1)
+				)
+			)
 		)
 	)
@@
 		(on_board yes)
 		(dnp no)
-		(property "Reference" "C226"
+		(property "Reference" "C15"
 			(at 83.058 158.75 90)
 			(effects
@@
 				)
 			)
+			(project "EE 447"
+				(path "/8dcae476-bf02-4dea-8567-670805b7ab7c/9f33d424-8f8c-499b-911f-2b5f72ba0270"
+					(reference "C15")
+					(unit 1)
+				)
+			)
 		)
 	)
@@
 		(on_board yes)
 		(dnp no)
-		(property "Reference" "U203"
+		(property "Reference" "U3"
 			(at 119.126 20.574 0)
 			(effects
@@
 				)
 			)
+			(project "EE 447"
+				(path "/8dcae476-bf02-4dea-8567-670805b7ab7c/9f33d424-8f8c-499b-911f-2b5f72ba0270"
+					(reference "U3")
+					(unit 1)
+				)
+			)
 		)
 	)
@@
 		(dnp no)
 		(fields_autoplaced yes)
-		(property "Reference" "R204"
+		(property "Reference" "R3"
 			(at 99.06 38.0999 0)
 			(effects
@@
 				)
 			)
+			(project "EE 447"
+				(path "/8dcae476-bf02-4dea-8567-670805b7ab7c/9f33d424-8f8c-499b-911f-2b5f72ba0270"
+					(reference "R3")
+					(unit 1)
+				)
+			)
 		)
 	)
@@
 		(dnp no)
 		(fields_autoplaced yes)
-		(property "Reference" "R206"
+		(property "Reference" "R6"
 			(at 113.03 54.6099 0)
 			(effects
@@
 				(path "/4d36fe0e-b49e-45a2-8e76-66c0323912e5"
 					(reference "R206")
+					(unit 1)
+				)
+			)
+			(project "EE 447"
+				(path "/8dcae476-bf02-4dea-8567-670805b7ab7c/9f33d424-8f8c-499b-911f-2b5f72ba0270"
+					(reference "R6")
 					(unit 1)
 				)
@@
 		(on_board yes)
 		(dnp no)
-		(property "Reference" "Q201"
+		(property "Reference" "Q1"
 			(at 55.88 34.2901 0)
 			(effects
@@
 				)
 			)
+			(project "EE 447"
+				(path "/8dcae476-bf02-4dea-8567-670805b7ab7c/9f33d424-8f8c-499b-911f-2b5f72ba0270"
+					(reference "Q1")
+					(unit 1)
+				)
+			)
 		)
 	)
@@
 		(on_board yes)
 		(dnp no)
-		(property "Reference" "C224"
+		(property "Reference" "C13"
 			(at 83.058 153.67 90)
 			(effects
@@
 				)
 			)
+			(project "EE 447"
+				(path "/8dcae476-bf02-4dea-8567-670805b7ab7c/9f33d424-8f8c-499b-911f-2b5f72ba0270"
+					(reference "C13")
+					(unit 1)
+				)
+			)
 		)
 	)
@@
 		(dnp no)
 		(fields_autoplaced yes)
-		(property "Reference" "C203"
+		(property "Reference" "C17"
 			(at 90.17 33.0199 0)
 			(effects
@@
 				)
 			)
+			(project "EE 447"
+				(path "/8dcae476-bf02-4dea-8567-670805b7ab7c/9f33d424-8f8c-499b-911f-2b5f72ba0270"
+					(reference "C17")
+					(unit 1)
+				)
+			)
 		)
 	)
@@
 		(dnp no)
 		(fields_autoplaced yes)
-		(property "Reference" "R202"
+		(property "Reference" "R2"
 			(at 29.21 26.67 90)
 			(effects
@@
 				)
 			)
+			(project "EE 447"
+				(path "/8dcae476-bf02-4dea-8567-670805b7ab7c/9f33d424-8f8c-499b-911f-2b5f72ba0270"
+					(reference "R2")
+					(unit 1)
+				)
+			)
 		)
 	)
@@
 		(dnp no)
 		(fields_autoplaced yes)
-		(property "Reference" "L201"
+		(property "Reference" "L1"
 			(at 43.18 45.72 90)
 			(effects
@@
 				)
 			)
+			(project "EE 447"
+				(path "/8dcae476-bf02-4dea-8567-670805b7ab7c/9f33d424-8f8c-499b-911f-2b5f72ba0270"
+					(reference "L1")
+					(unit 1)
+				)
+			)
 		)
 	)
@@
 		(dnp no)
 		(fields_autoplaced yes)
-		(property "Reference" "D201"
+		(property "Reference" "D1"
 			(at 28.8925 58.42 0)
 			(effects
@@
 					(unit 1)
 				)
+			)
+			(project "EE 447"
+				(path "/8dcae476-bf02-4dea-8567-670805b7ab7c/9f33d424-8f8c-499b-911f-2b5f72ba0270"
+					(reference "D1")
+					(unit 1)
+				)

Commit message: added pinheader
Parts:
- added J9: 61302421121, Custom:61302421121, symbol 61302421121:61302421121
Connections:
- net 3V3_OUT: now also J9.16
- net BS: now also J9.18, J9.7
- net EPD_BUSY: now also J9.10
- net EPD_CS: now also J9.11
- net EPD_DC: now also J9.12
- net EPD_DIN: now also J9.13
- net EPD_RST: now also J9.9
- net EPD_SCK: now also J9.14
- net GDR: now also J9.1
- net RESE: now also J9.4
- net VGH: now also J9.22
- net VGL: now also J9.24
- net SUB18: now reaches C11.1, J2.18
- net SUB18: now also J9.17
- net SUB20: now reaches C12.1, J2.20
- net SUB20: now also J9.19
- net SUB22: now reaches C14.1, J2.22
- net SUB22: now also J9.21
- net SUB24: now reaches C16.1, J2.24
- net SUB24: now also J9.23
- net SUB5: now reaches C9.1, J2.5
- net SUB5: now also J9.6

Commit message: i added stuff
Connections:
- net VCC is gone; now on net 3V3_OUT: U3.3
- net BS renamed GND
- net EPD_DIN renamed MOSI
- net EPD_SCK renamed CLK
- net VCC_INT renamed +3.3V
Changed lines of the file:
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@@
 	(paper "A4")
 	(junction
+		(at 86.36 26.67)
+		(diameter 0)
+		(color 0 0 0 0)
+	)
+	(junction
 		(at 21.59 33.02)
 		(diameter 0)
@@
 	(wire
 		(pts
-			(xy 86.36 26.67) (xy 86.36 30.48)
-		)
-		(stroke
-			(width 0)
-			(type default)
-		)
-	)
-	(wire
-		(pts
 			(xy 33.02 50.8) (xy 36.83 50.8)
 		)
@@
 	(wire
 		(pts
-			(xy 53.34 133.35) (xy 60.96 133.35)
+			(xy 53.34 133.35) (xy 73.66 133.35)
 		)
 		(stroke
@@
 	(wire
 		(pts
+			(xy 86.36 21.59) (xy 86.36 26.67)
+		)
+		(stroke
+			(width 0)
+			(type default)
+		)
+	)
+	(wire
+		(pts
 			(xy 53.34 140.97) (xy 60.96 140.97)
 		)
@@
 	(wire
 		(pts
-			(xy 53.34 135.89) (xy 60.96 135.89)
+			(xy 53.34 135.89) (xy 73.66 135.89)
 		)
 		(stroke
@@
 	(wire
 		(pts
+			(xy 86.36 26.67) (xy 86.36 30.48)
+		)
+		(stroke
+			(width 0)
+			(type default)
+		)
+	)
+	(wire
+		(pts
 			(xy 53.34 158.75) (xy 71.12 158.75)
 		)
@@
 		)
 	)
-	(label "VCC"
-		(at 127 26.67 0)
-		(effects
-			(font
-				(size 1.27 1.27)
-			)
-			(justify left bottom)
-		)
-	)
 	(label "RESE"
 		(at 46.99 22.86 0)
@@
 		)
 	)
-	(label "VCC_INT"
-		(at 86.36 26.67 0)
-		(effects
-			(font
-				(size 1.27 1.27)
-			)
-			(justify left bottom)
-		)
-	)
 	(label "GND"
 		(at 127 60.96 0)
@@
 		)
 	)
-	(label "VCC"
-		(at 127 26.67 0)
-		(effects
-			(font
-				(size 1.27 1.27)
-			)
-			(justify left bottom)
-		)
-	)
 	(label "VGH"
 		(at 52.07 83.82 0)
@@
 		)
 	)
-	(label "VCC"
-		(at 127 26.67 0)
-		(effects
-			(font
-				(size 1.27 1.27)
-			)
-			(justify left bottom)
-		)
-	)
 	(label "RESE"
 		(at 46.99 22.86 0)
@@
 		)
 	)
-	(label "VCC"
-		(at 127 26.67 0)
+	(label "SUB20"
+		(at 111.76 134.62 0)
 		(effects
 			(font
@@
 		)
 	)
-	(label "SUB20"
-		(at 111.76 134.62 0)
+	(label "EPD_BUSY"
+		(at 149.86 121.92 0)
 		(effects
 			(font
@@
 		)
 	)
-	(label "EPD_BUSY"
-		(at 149.86 121.92 0)
+	(label "3V3_OUT"
+		(at 130.81 26.67 0)
 		(effects
 			(font
@@
 		)
 	)
-	(label "VCC_INT"
-		(at 86.36 26.67 0)
-		(effects
-			(font
-				(size 1.27 1.27)
-			)
-			(justify left bottom)
-		)
-	)
 	(label "EPD_PWR"
 		(at 86.36 48.26 0)
@@
 		)
 	)
-	(label "VCC_INT"
-		(at 86.36 26.67 0)
+	(label "GND"
+		(at 16.51 43.18 0)
 		(effects
 			(font
@@
 		)
 	)
-	(label "GND"
-		(at 16.51 43.18 0)
+	(label "EPD_DIN"
+		(at 111.76 127 0)
 		(effects
 			(font
@@
 		)
 	)
-	(label "VCC_INT"
-		(at 86.36 26.67 0)
+	(label "SUB5"
+		(at 60.96 113.03 0)
 		(effects
 			(font
@@
 	)
 	(label "EPD_DIN"
-		(at 111.76 127 0)
+		(at 60.96 135.89 0)
 		(effects
 			(font
@@
 		)
 	)
-	(label "SUB5"
-		(at 60.96 113.03 0)
+	(global_label "MOSI"
+		(shape input)
+		(at 73.66 135.89 0)
+		(fields_autoplaced yes)
 		(effects
 			(font
 				(size 1.27 1.27)
 			)
-			(justify left bottom)
+			(justify left)
+		)
+		(property "Intersheetrefs" "${INTERSHEET_REFS}"
+			(at 81.2414 135.89 0)
+			(effects
+				(font
+					(size 1.27 1.27)
+				)
+				(justify left)
+				(hide yes)
+			)
 		)
 	)
-	(label "EPD_DIN"
-		(at 60.96 135.89 0)
+	(global_label "CLK"
+		(shape input)
+		(at 73.66 133.35 0)
+		(fields_autoplaced yes)
 		(effects
 			(font
 				(size 1.27 1.27)
 			)
-			(justify left bottom)
+			(justify left)
+		)
+		(property "Intersheetrefs" "${INTERSHEET_REFS}"
+			(at 80.2133 133.35 0)
+			(effects
+				(font
+					(size 1.27 1.27)
+				)
+				(justify left)
+				(hide yes)
+			)
 		)
 	)
@@
 	)
 	(symbol
+		(lib_id "power:GND")
+		(at 16.51 43.18 0)
+		(unit 1)
+		(exclude_from_sim no)
+		(in_bom yes)
+		(on_board yes)
+		(dnp no)
+		(fields_autoplaced yes)
+		(property "Reference" "#PWR0101"
+			(at 16.51 49.53 0)
+			(effects
+				(font
+					(size 1.27 1.27)
+				)
+				(hide yes)
+			)
+		)
+		(property "Value" "GND"
+			(at 16.51 48.26 0)
+			(effects
+				(font
+					(size 1.27 1.27)
+				)
+			)
+		)
+		(property "Footprint" ""
+			(at 16.51 43.18 0)
+			(effects
+				(font
+					(size 1.27 1.27)
+				)
+				(hide yes)
+			)
+		)
+		(property "Datasheet" ""
+			(at 16.51 43.18 0)
+			(effects
+				(font
+					(size 1.27 1.27)
+				)
+				(hide yes)
+			)
+		)
+		(property "Description" "Power symbol creates a global label with name \"GND\" , ground"
+			(at 16.51 43.18 0)
+			(effects
+				(font
+					(size 1.27 1.27)
+				)
+				(hide yes)
+			)
+		)
+		(pin "1"
+		)
+		(instances
+			(project ""
+				(path "/4d36fe0e-b49e-45a2-8e76-66c0323912e5"
+					(reference "#PWR01")
+					(unit 1)
+				)
+			)
+			(project "EE 447"
+				(path "/8dcae476-bf02-4dea-8567-670805b7ab7c/9f33d424-8f8c-499b-911f-2b5f72ba0270"
+					(reference "#PWR0101")
+					(unit 1)
+				)
+			)
+		)
+	)
+	(symbol
 		(lib_id "Device:R")
 		(at 96.52 39.37 0)
@@
 					(unit 1)
 				)
+			)
+		)
+	)
+	(symbol
+		(lib_id "power:+3.3V")
+		(at 86.36 21.59 0)
+		(unit 1)
+		(exclude_from_sim no)
+		(in_bom yes)
+		(on_board yes)
+		(dnp no)
+		(fields_autoplaced yes)
+		(property "Reference" "#PWR0102"
+			(at 86.36 25.4 0)
+			(effects
+				(font
+					(size 1.27 1.27)
+				)
+				(hide yes)
+			)
+		)
+		(property "Value" "+3.3V"
+			(at 86.36 16.51 0)
+			(effects
+				(font
+					(size 1.27 1.27)
+				)
+			)
+		)
+		(property "Footprint" ""
+			(at 86.36 21.59 0)
+			(effects
+				(font
+					(size 1.27 1.27)
+				)
+				(hide yes)
+			)
+		)
+		(property "Datasheet" ""
+			(at 86.36 21.59 0)
+			(effects
+				(font
+					(size 1.27 1.27)
+				)
+				(hide yes)
+			)
+		)
+		(property "Description" "Power symbol creates a global label with name \"+3.3V\""
+			(at 86.36 21.59 0)
+			(effects
+				(font
+					(size 1.27 1.27)
+				)
+				(hide yes)
+			)
+		)
+		(pin "1"
+		)
+		(instances
+			(project ""
+				(path "/4d36fe0e-b49e-45a2-8e76-66c0323912e5"
+					(reference "#PWR02")
+					(unit 1)
+				)
+			)
+			(project "EE 447"
+				(path "/8dcae476-bf02-4dea-8567-670805b7ab7c/9f33d424-8f8c-499b-911f-2b5f72ba0270"
+					(reference "#PWR0102")
+					(unit 1)
+				)
