File: PCB_June/PCB.kicad_sch (KiCad schematic)
At the start: 26 parts, among them J2 FH34SRJ-24S-0.5SH_99_, J9 61302421121, Q1 BSS138, Q2 S8050, U3 AO3401

Commit message: footprint pull push
Parts:
- removed D1, D2, D3: MBR0530, Diode_SMD:D_SOD-123, symbol Diode:MBR0530
- added CR1, CR2, CR3: SS0530_R1_00001, Library:SOD-123_PNJ, symbol SymbolLibrary:SS0530_R1_00001
Connections:
- net GND: now also CR3.1
- net VGH: now also CR1.1
- net VGL: now also CR2.2
- net at C8.2, L1.2, Q1.3 (D): now also CR1.2
- net at C8.1: now also CR2.1, CR3.2
Changed lines of the file:
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@@
 	(wire
 		(pts
-			(xy 36.83 77.47) (xy 36.83 83.82)
-		)
-		(stroke
-			(width 0)
-			(type default)
-		)
-	)
-	(wire
-		(pts
 			(xy 107.95 26.67) (xy 107.95 29.21)
 		)
@@
 	(wire
 		(pts
-			(xy 21.59 64.77) (xy 25.4 64.77)
+			(xy 21.59 64.77) (xy 24.13 64.77)
 		)
 		(stroke
@@
 	(wire
 		(pts
-			(xy 33.02 64.77) (xy 36.83 64.77)
-		)
-		(stroke
-			(width 0)
-			(type default)
-		)
-	)
-	(wire
-		(pts
 			(xy 34.29 41.91) (xy 34.29 50.8)
 		)
@@
 	(wire
 		(pts
-			(xy 52.07 77.47) (xy 52.07 83.82)
+			(xy 52.07 80.01) (xy 52.07 83.82)
 		)
 		(stroke
@@
 	(wire
 		(pts
+			(xy 34.29 64.77) (xy 36.83 64.77)
+		)
+		(stroke
+			(width 0)
+			(type default)
+		)
+	)
+	(wire
+		(pts
+			(xy 36.83 80.01) (xy 36.83 83.82)
+		)
+		(stroke
+			(width 0)
+			(type default)
+		)
+	)
+	(wire
+		(pts
 			(xy 96.52 26.67) (xy 107.95 26.67)
 		)
@@
 	)
 	(symbol
-		(lib_id "Diode:MBR0530")
-		(at 52.07 73.66 90)
-		(unit 1)
-		(exclude_from_sim no)
-		(in_bom yes)
-		(on_board yes)
-		(dnp no)
-		(property "Reference" "D3"
-			(at 57.404 72.898 90)
-			(effects
-				(font
-					(size 1.27 1.27)
-				)
-				(justify right)
-			)
-		)
-		(property "Value" "MBR0530"
-			(at 54.356 74.3586 90)
-			(effects
-				(font
-					(size 1.27 1.27)
-				)
-				(justify right)
-			)
-		)
-		(property "Footprint" "Diode_SMD:D_SOD-123"
-			(at 56.515 73.66 0)
-			(effects
-				(font
-					(size 1.27 1.27)
-				)
-				(hide yes)
-			)
-		)
-		(property "Datasheet" "http://www.mccsemi.com/up_pdf/MBR0520~MBR0580(SOD123).pdf"
-			(at 52.07 73.66 0)
-			(effects
-				(font
-					(size 1.27 1.27)
-				)
-				(hide yes)
-			)
-		)
-		(property "Description" "30V 0.5A Schottky Power Rectifier Diode, SOD-123"
-			(at 52.07 73.66 0)
-			(effects
-				(font
-					(size 1.27 1.27)
-				)
-				(hide yes)
-			)
-		)
-		(pin "1"
-		)
-		(pin "2"
-		)
-		(instances
-			(project ""
-				(path "/4d36fe0e-b49e-45a2-8e76-66c0323912e5"
-					(reference "D203")
-					(unit 1)
-				)
-			)
-			(project "EE 447"
-				(path "/8dcae476-bf02-4dea-8567-670805b7ab7c/9f33d424-8f8c-499b-911f-2b5f72ba0270"
-					(reference "D3")
-					(unit 1)
-				)
-			)
-		)
-	)
-	(symbol
 		(lib_id "Device:C")
 		(at 74.93 146.05 90)
@@
 	)
 	(symbol
-		(lib_id "Diode:MBR0530")
-		(at 36.83 73.66 270)
+		(lib_id "SymbolLibrary:SS0530_R1_00001")
+		(at 52.07 69.85 270)
 		(unit 1)
 		(exclude_from_sim no)
@@
 		(dnp no)
 		(fields_autoplaced yes)
-		(property "Reference" "D2"
-			(at 39.37 72.0724 90)
+		(property "Reference" "CR1"
+			(at 55.88 73.6599 90)
 			(effects
 				(font
-					(size 1.27 1.27)
+					(size 1.524 1.524)
 				)
 				(justify left)
 			)
 		)
-		(property "Value" "MBR0530"
-			(at 39.37 74.6124 90)
+		(property "Value" "SS0530_R1_00001"
+			(at 55.88 76.1999 90)
 			(effects
 				(font
-					(size 1.27 1.27)
+					(size 1.524 1.524)
 				)
 				(justify left)
 			)
 		)
-		(property "Footprint" "Diode_SMD:D_SOD-123"
-			(at 32.385 73.66 0)
+		(property "Footprint" "Library:SOD-123_PNJ"
+			(at 52.07 69.85 0)
 			(effects
 				(font
 					(size 1.27 1.27)
+					(italic yes)
 				)
 				(hide yes)
 			)
 		)
-		(property "Datasheet" "http://www.mccsemi.com/up_pdf/MBR0520~MBR0580(SOD123).pdf"
-			(at 36.83 73.66 0)
+		(property "Datasheet" "SS0530_R1_00001"
+			(at 52.07 69.85 0)
 			(effects
 				(font
 					(size 1.27 1.27)
+					(italic yes)
 				)
 				(hide yes)
 			)
 		)
-		(property "Description" "30V 0.5A Schottky Power Rectifier Diode, SOD-123"
-			(at 36.83 73.66 0)
+		(property "Description" ""
+			(at 52.07 69.85 0)
 			(effects
 				(font
@@
 		(instances
 			(project ""
-				(path "/4d36fe0e-b49e-45a2-8e76-66c0323912e5"
-					(reference "D202")
-					(unit 1)
-				)
-			)
-			(project "EE 447"
 				(path "/8dcae476-bf02-4dea-8567-670805b7ab7c/9f33d424-8f8c-499b-911f-2b5f72ba0270"
-					(reference "D2")
+					(reference "CR1")
 					(unit 1)
 				)
@@
 	)
 	(symbol
+		(lib_id "SymbolLibrary:SS0530_R1_00001")
+		(at 36.83 80.01 90)
+		(unit 1)
+		(exclude_from_sim no)
+		(in_bom yes)
+		(on_board yes)
+		(dnp no)
+		(property "Reference" "CR2"
+			(at 40.64 73.6599 90)
+			(effects
+				(font
+					(size 1.524 1.524)
+				)
+				(justify right)
+			)
+		)
+		(property "Value" "SS0530_R1_00001"
+			(at 33.274 71.374 0)
+			(effects
+				(font
+					(size 1.524 1.524)
+				)
+				(justify right)
+			)
+		)
+		(property "Footprint" "Library:SOD-123_PNJ"
+			(at 36.83 80.01 0)
+			(effects
+				(font
+					(size 1.27 1.27)
+					(italic yes)
+				)
+				(hide yes)
+			)
+		)
+		(property "Datasheet" "SS0530_R1_00001"
+			(at 36.83 80.01 0)
+			(effects
+				(font
+					(size 1.27 1.27)
+					(italic yes)
+				)
+				(hide yes)
+			)
+		)
+		(property "Description" ""
+			(at 36.83 80.01 0)
+			(effects
+				(font
+					(size 1.27 1.27)
+				)
+				(hide yes)
+			)
+		)
+		(pin "1"
+		)
+		(pin "2"
+		)
+		(instances
+			(project ""
+				(path "/8dcae476-bf02-4dea-8567-670805b7ab7c/9f33d424-8f8c-499b-911f-2b5f72ba0270"
+					(reference "CR2")
+					(unit 1)
+				)
+			)
+		)
+	)
+	(symbol
 		(lib_id "Transistor_FET:BSS138")
 		(at 49.53 33.02 0)
@@
 	)
 	(symbol
-		(lib_id "Diode:MBR0530")
-		(at 29.21 64.77 0)
+		(lib_id "SymbolLibrary:SS0530_R1_00001")
+		(at 34.29 64.77 180)
 		(unit 1)
 		(exclude_from_sim no)
@@
 		(on_board yes)
 		(dnp no)
-		(fields_autoplaced yes)
-		(property "Reference" "D1"
-			(at 28.8925 58.42 0)
+		(property "Reference" "CR3"
+			(at 29.21 58.42 0)
 			(effects
 				(font
-					(size 1.27 1.27)
+					(size 1.524 1.524)
 				)
 			)
 		)
-		(property "Value" "MBR0530"
-			(at 28.8925 60.96 0)
+		(property "Value" "SS0530_R1_00001"
+			(at 29.21 60.96 0)
 			(effects
 				(font
-					(size 1.27 1.27)
+					(size 1.524 1.524)
 				)
 			)
 		)
-		(property "Footprint" "Diode_SMD:D_SOD-123"
-			(at 29.21 69.215 0)
+		(property "Footprint" "Library:SOD-123_PNJ"
+			(at 34.29 64.77 0)
 			(effects
 				(font
 					(size 1.27 1.27)
+					(italic yes)
 				)
 				(hide yes)
 			)
 		)
-		(property "Datasheet" "http://www.mccsemi.com/up_pdf/MBR0520~MBR0580(SOD123).pdf"
-			(at 29.21 64.77 0)
+		(property "Datasheet" "SS0530_R1_00001"
+			(at 34.29 64.77 0)
 			(effects
 				(font
 					(size 1.27 1.27)
+					(italic yes)
 				)
 				(hide yes)
 			)
 		)
-		(property "Description" "30V 0.5A Schottky Power Rectifier Diode, SOD-123"
-			(at 29.21 64.77 0)
+		(property "Description" ""
+			(at 34.29 64.77 0)
 			(effects
 				(font
@@
 			)
 		)
-		(pin "2"
-		)
 		(pin "1"
 		)
+		(pin "2"
+		)
 		(instances
 			(project ""
-				(path "/4d36fe0e-b49e-45a2-8e76-66c0323912e5"
-					(reference "D201")
-					(unit 1)
-				)
-			)
-			(project "EE 447"
 				(path "/8dcae476-bf02-4dea-8567-670805b7ab7c/9f33d424-8f8c-499b-911f-2b5f72ba0270"
-					(reference "D1")
+					(reference "CR3")
 					(unit 1)
 				)

Commit message: eieio i think i done
Parts:
- U3: value AO3401 -> PJA3401A; footprint Custom:SOT23 -> Package_TO_SOT_SMD:SOT-23
Changed lines of the file:
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@@
 			)
 		)
-		(property "Datasheet" "~"
+		(property "Datasheet" "https://www.digikey.com/en/products/detail/littelfuse-inc/WSTM0805QLR470FNR/18795427"
 			(at 29.21 22.86 0)
 			(effects
@@
 			)
 		)
-		(property "Datasheet" "~"
+		(property "Datasheet" "https://www.digikey.com/en/products/detail/stackpole-electronics-inc/RMCF0805JT47K0/1757842"
 			(at 107.95 33.02 0)
 			(effects
@@
 			)
 		)
-		(property "Datasheet" "https://componentsearchengine.com/Datasheets/1/61302421121.pdf"
+		(property "Datasheet" "https://www.mouser.com/ProductDetail/Wurth-Elektronik/61302421121?qs=PhR8RmCirEZkViXMpcFdWg%3D%3D&srsltid=AfmBOop_fFQ2_g8Ld3pw2KMKNhrAhxI88sAUzXO9IHa7Qle_StAjma5G"
 			(at 138.43 306.68 0)
 			(effects
@@
 			)
 		)
-		(property "Datasheet" "SS0530_R1_00001"
+		(property "Datasheet" "https://www.digikey.com/en/products/detail/panjit-international-inc/SS0530-R1-00001/14660025"
 			(at 52.07 69.85 0)
 			(effects
@@
 			)
 		)
-		(property "Datasheet" "http://www.unisonic.com.tw/datasheet/S8050.pdf"
+		(property "Datasheet" "https://www.digikey.com/en/products/detail/umw/S8050/17635323"
 			(at 119.38 48.26 0)
 			(effects
@@
 			)
 		)
-		(property "Value" "AO3401"
+		(property "Value" "PJA3401A"
 			(at 119.38 22.86 0)
 			(effects
@@
 			)
 		)
-		(property "Footprint" "Custom:SOT23"
+		(property "Footprint" "Package_TO_SOT_SMD:SOT-23"
 			(at 121.92 26.67 0)
 			(effects
@@
 			)
 		)
-		(property "Datasheet" ""
+		(property "Datasheet" "https://www.mouser.com/ProductDetail/Panjit/PJA3401A_R1_00001?qs=sPbYRqrBIVk%2F%252BjzjJws01Q%3D%3D&srsltid=AfmBOoppGGn4NUPxGcch7cElXr9U5cPY8zTJL7fS2APxaADN3IHJET62"
 			(at 121.92 26.67 0)
 			(effects
@@
 			)
 		)
-		(property "Datasheet" "~"
+		(property "Datasheet" "https://www.digikey.com/en/products/detail/stackpole-electronics-inc/RMCF0805JT47K0/1757842"
 			(at 96.52 39.37 0)
 			(effects
@@
 			)
 		)
-		(property "Datasheet" "SS0530_R1_00001"
+		(property "Datasheet" "https://www.digikey.com/en/products/detail/panjit-international-inc/SS0530-R1-00001/14660025"
 			(at 36.83 80.01 0)
 			(effects
@@
 			)
 		)
-		(property "Datasheet" "SS0530_R1_00001"
+		(property "Datasheet" "https://www.digikey.com/en/products/detail/panjit-international-inc/SS0530-R1-00001/14660025"
 			(at 34.29 64.77 0)
 			(effects

Commit message: small fixes
Changed lines of the file:
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@@
 					(size 1.27 1.27)
 				)
+				(hide yes)
 			)
 		)

Commit message: sdfghjk
Parts:
- Q2: footprint Package_TO_SOT_THT:TO-92_Inline -> Package_TO_SOT_SMD:SOT-23_Handsoldering
Changed lines of the file:
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@@
 			)
 		)
-		(property "Footprint" "Package_TO_SOT_THT:TO-92_Inline"
+		(property "Footprint" "Package_TO_SOT_SMD:SOT-23_Handsoldering"
 			(at 124.46 50.165 0)
 			(effects
@@
 			)
 		)
-		(property "Datasheet" "https://www.digikey.com/en/products/detail/onsemi/BSS138/244210"
+		(property "Datasheet" "https://www.mouser.com/ProductDetail/onsemi-Fairchild/BSS138?qs=HK%252BeIG1iaahCeqBvjB4arg%3D%3D&srsltid=AfmBOoqSNHRxNY05tuDQ32Q_ya6yO_gO9lrnV_3A-Ol45sM-SCPd4I5t"
 			(at 54.61 29.21 0)
 			(effects

Commit message: bjt
Parts:
- removed Q2: S8050, Package_TO_SOT_SMD:SOT-23_Handsoldering, symbol Transistor_BJT:S8050
- added Q2: SMD-TRANSISTORS-NPN-25V-500MW_SOT-23_, Library:S8050_SOT-23, symbol SymbolLibrary:SMD-TRANSISTORS-NPN-25V-500MW_SOT-23_
Connections:
- net GND: now also Q2.2
- net at R5.2, U3.1: now also Q2.3
- net at R4.1, R6.2: now also Q2.1
Changed lines of the file:
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@@
 	(wire
 		(pts
-			(xy 110.49 48.26) (xy 114.3 48.26)
+			(xy 110.49 48.26) (xy 116.84 48.26)
 		)
 		(stroke
@@
 	)
 	(symbol
+		(lib_id "SymbolLibrary:SMD-TRANSISTORS-NPN-25V-500MW_SOT-23_")
+		(at 119.38 48.26 0)
+		(unit 1)
+		(exclude_from_sim no)
+		(in_bom yes)
+		(on_board yes)
+		(dnp no)
+		(fields_autoplaced yes)
+		(property "Reference" "Q2"
+			(at 123.19 46.9441 0)
+			(effects
+				(font
+					(size 1.27 1.27)
+				)
+				(justify left)
+			)
+		)
+		(property "Value" "SMD-TRANSISTORS-NPN-25V-500MW_SOT-23_"
+			(at 123.19 49.4841 0)
+			(effects
+				(font
+					(size 1.27 1.27)
+				)
+				(justify left)
+			)
+		)
+		(property "Footprint" "Library:S8050_SOT-23"
+			(at 119.38 48.26 0)
+			(effects
+				(font
+					(size 1.27 1.27)
+				)
+				(justify bottom)
+				(hide yes)
+			)
+		)
+		(property "Datasheet" ""
+			(at 119.38 48.26 0)
+			(effects
+				(font
+					(size 1.27 1.27)
+				)
+				(hide yes)
+			)
+		)
+		(property "Description" ""
+			(at 119.38 48.26 0)
+			(effects
+				(font
+					(size 1.27 1.27)
+				)
+				(hide yes)
+			)
+		)
+		(property "MF" "UMW"
+			(at 119.38 48.26 0)
+			(effects
+				(font
+					(size 1.27 1.27)
+				)
+				(justify bottom)
+				(hide yes)
+			)
+		)
+		(property "Description_1" "Bipolar (BJT) Transistor NPN 25 V 500 mA 150MHz 300 mW Surface Mount SOT-23"
+			(at 119.38 48.26 0)
+			(effects
+				(font
+					(size 1.27 1.27)
+				)
+				(justify bottom)
+				(hide yes)
+			)
+		)
+		(property "Package" "None"
+			(at 119.38 48.26 0)
+			(effects
+				(font
+					(size 1.27 1.27)
+				)
+				(justify bottom)
+				(hide yes)
+			)
+		)
+		(property "MPN" "S8050"
+			(at 119.38 48.26 0)
+			(effects
+				(font
+					(size 1.27 1.27)
+				)
+				(justify bottom)
+				(hide yes)
+			)
+		)
+		(property "Price" "None"
+			(at 119.38 48.26 0)
+			(effects
+				(font
+					(size 1.27 1.27)
+				)
+				(justify bottom)
+				(hide yes)
+			)
+		)
+		(property "SnapEDA_Link" "https://www.snapeda.com/parts/S8050/UMW/view-part/?ref=snap"
+			(at 119.38 48.26 0)
+			(effects
+				(font
+					(size 1.27 1.27)
+				)
+				(justify bottom)
+				(hide yes)
+			)
+		)
+		(property "MP" "S8050"
+			(at 119.38 48.26 0)
+			(effects
+				(font
+					(size 1.27 1.27)
+				)
+				(justify bottom)
+				(hide yes)
+			)
+		)
+		(property "Availability" "In Stock"
+			(at 119.38 48.26 0)
+			(effects
+				(font
+					(size 1.27 1.27)
+				)
+				(justify bottom)
+				(hide yes)
+			)
+		)
+		(property "Check_prices" "https://www.snapeda.com/parts/S8050/UMW/view-part/?ref=eda"
+			(at 119.38 48.26 0)
+			(effects
+				(font
+					(size 1.27 1.27)
+				)
+				(justify bottom)
+				(hide yes)
+			)
+		)
+		(pin "3"
+		)
+		(pin "1"
+		)
+		(pin "2"
+		)
+		(instances
+			(project ""
+				(path "/8dcae476-bf02-4dea-8567-670805b7ab7c/9f33d424-8f8c-499b-911f-2b5f72ba0270"
+					(reference "Q2")
+					(unit 1)
+				)
+			)
+		)
+	)
+	(symbol
 		(lib_id "Device:C")
 		(at 74.93 161.29 90)
@@
 					(unit 1)
 				)
-			)
-		)
-	)
-	(symbol
-		(lib_id "Transistor_BJT:S8050")
-		(at 119.38 48.26 0)
-		(unit 1)
-		(exclude_from_sim no)
-		(in_bom yes)
-		(on_board yes)
-		(dnp no)
-		(fields_autoplaced yes)
-		(property "Reference" "Q2"
-			(at 124.46 46.9899 0)
-			(effects
-				(font
-					(size 1.27 1.27)
-				)
-				(justify left)
-			)
-		)
-		(property "Value" "S8050"
-			(at 124.46 49.5299 0)
-			(effects
-				(font
-					(size 1.27 1.27)
-				)
-				(justify left)
-			)
-		)
-		(property "Footprint" "Package_TO_SOT_SMD:SOT-23_Handsoldering"
-			(at 124.46 50.165 0)
-			(effects
-				(font
-					(size 1.27 1.27)
-					(italic yes)
-				)
-				(justify left)
-				(hide yes)
-			)
-		)
-		(property "Datasheet" "https://www.digikey.com/en/products/detail/umw/S8050/17635323"
-			(at 119.38 48.26 0)
-			(effects
-				(font
-					(size 1.27 1.27)
-				)
-				(justify left)
-				(hide yes)
-			)
-		)
-		(property "Description" "0.7A Ic, 20V Vce, Low Voltage High Current NPN Transistor, TO-92"
-			(at 119.38 48.26 0)
-			(effects
-				(font
-					(size 1.27 1.27)
-				)
-				(hide yes)
-			)
-		)
-		(pin "2"
-		)
-		(pin "3"
-		)
-		(pin "1"
-		)
-		(instances
-			(project ""
-				(path "/4d36fe0e-b49e-45a2-8e76-66c0323912e5"
-					(reference "Q202")
-					(unit 1)
-				)
-			)
-			(project "EE 447"
-				(path "/8dcae476-bf02-4dea-8567-670805b7ab7c/9f33d424-8f8c-499b-911f-2b5f72ba0270"
-					(reference "Q2")
-					(unit 1)
-				)

Commit message: checked DRC but check again ig, i checked all my footprint
 i made a small change connecting 15 and 16
Connections:
- net 3V3_OUT: now also J9.15
- no-connect marks 11 -> 10
Changed lines of the file:
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@@
-	)
-	(no_connect
-		(at 119.38 129.54)
 	)
 	(no_connect
@@
 	(wire
 		(pts
+			(xy 111.76 129.54) (xy 119.38 129.54)
+		)
+		(stroke
+			(width 0)
+			(type default)
+		)
+	)
+	(wire
+		(pts
 			(xy 34.29 50.8) (xy 35.56 50.8)
 		)
@@
 		(effects
 			(font
+				(size 1.27 1.27)
+			)
+			(justify left bottom)
+		)
+	)
+	(label "3V3_OUT"
+		(at 111.76 129.54 0)
+		(effects
+			(font
