File: PCB_power/power/power.kicad_sch (KiCad schematic)
At the start: 39 parts, among them J3 S2B-PH-K-SLFSN, J4 Conn_01x01_Pin, J5 Conn_01x02_Pin, J6 Conn_01x01_Pin, J7 Conn_01x01_Pin, J8 Conn_01x02_Pin, Q3 DMG3415UQ-7, SW1 SLW-121586-5A-D, U4 LM66100DCK, U5 BQ21040DBV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

Commit message: added back annotations
Other:
- note added: "IOUT = KISET / RISET IOUT = 540 / 5.36k = 0.1A"
- note added: "To Disable the temp sense function, use a fixed 10k resistor between the TS (terminal 1) and Vss"
Changed lines of the file:
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@@
+		)
+	)
+	(text "To Disable the temp sense function, \nuse a fixed 10k resistor between the \nTS (terminal 1) and Vss"
+		(exclude_from_sim no)
+		(at 79.756 84.328 0)
+		(effects
+			(font
+				(size 1.27 1.27)
+			)
+			(justify left)
 		)
 	)
@@
 			)
 		)
+	)
+	(text "IOUT = KISET / RISET\nIOUT = 540 / 5.36k = 0.1A\n"
+		(exclude_from_sim no)
+		(at 48.006 84.074 0)
+		(effects
+			(font
+				(size 1.27 1.27)
+			)
+		)
